File: SRSFC.kicad_sch (KiCad schematic)
At the start: 46 parts, among them J1 SWD_interface, X1 25MHz

Commit message: added BMP388
Parts:
- added C27: .1uF, Capacitor_SMD:C_0402_1005Metric, symbol Device:C
- added C28: 100nF, Capacitor_SMD:C_0402_1005Metric, symbol Device:C
- added CARD1: ~, SD_CARD_READER:TF-SMD_TF-PUSH, symbol SD_CARD_READER:TF PUSH
- added U6: ~, BMP388:SENSORM-SMD_BMP388, symbol BMP388:BMP388
Connections:
- net +3.3V: now also C27.2, C28.1, CARD1.4 (VDD), U6.1 (VDDIO), U6.10 (VDD)
- net GND: now also C27.1, C28.2, CARD1.CD, U6.3 (VSS), U6.8 (VSS), U6.9 (VSS)
- net SDIO_D0: now reaches U1.65 (PC8)
- net SDIO_D0: now also CARD1.7 (DAT0)
- net SDIO_D1: now reaches U1.66 (PC9)
- net SDIO_D1: now also CARD1.8 (DAT1)
- net SDIO_D2: now reaches U1.78 (PC10)
- net SDIO_D2: now also CARD1.2 (CD/DAT3)
- net SDIO_D3: now reaches U1.79 (PC11)
- net SDIO_D3: now also CARD1.3 (CMD)
- net SDIO_SCK: now reaches U1.80 (PC12)
- net SDIO_SCK: now also CARD1.5 (CLX)
- net SDIO_CMD: now reaches U1.83 (PD2)
- net SDIO_CMD: now also CARD1.6 (VSS)
Other:
- moved on the sheet: C18, C20, U3
